Commit message: ros_MP & description

File: description/description/urdf/description.urdf (robot description, URDF)
Before this commit: robot description, 8 links, 7 joints
Links:
- removed link caster_link
- removed link imu_base
- removed link usb_cam
- removed link wheel_L_link
- removed link wheel_R_link
- added link camera_link, mass 0.084224; collision mesh filename=package://description/meshes/camera_link.STL; visual mesh filename=package://description/meshes/camera_link.STL
- link base_link: mass 0.519076841043834 -> 5.6969
- link lidar_link: mass 0.090366 -> 0.18368
Joints:
- removed joint cam_joint
- removed joint caster_joint
- removed joint imu_joint
- removed joint wheel_L_joint
- removed joint wheel_R_joint
- added joint camera_joint: type fixed, parent base_link, child camera_link, origin xyz=-0.056159 -0.069676 0.34735 rpy=1.5478 0 0, axis 0 0 0
- joint lidar_joint: origin xyz=0.0042092 0.080995 0.1932 rpy=3.14 -3.14 1.57 -> xyz=0.00072357 -0.084809 0.1763 rpy=0 0 0

Commit message: 2021.08.16

File: description/description/urdf/description.urdf (robot description, URDF)
Before this commit: robot description, 4 links, 3 joints
Joints:
- joint base_joint: origin xyz=0.0 0.0 0 rpy=0 0 -1.57 -> xyz=0.0 0.0 0 rpy=0 0 1.57
- joint lidar_joint: origin xyz=0.00072357 -0.084809 0.1763 rpy=0 0 0 -> xyz=0.00072357 -0.084809 0.1763 rpy=0 3.14 1.57

Commit message: raspi

File: description/description/urdf/description.urdf (robot description, URDF)
Before this commit: robot description, 4 links, 3 joints
Joints:
- joint lidar_joint: origin xyz=0.00072357 -0.084809 0.1763 rpy=0 3.14 1.57 -> xyz=0.00072357 -0.084809 0.1763 rpy=0 0 -1.57
